Commit message: updated usv urdf

File: utils/vrx/x_drive/component_config.xacro (robot description, xacro)
@@ -14,4 +14,6 @@
     <!-- === wamv_ball_shooter === -->
       <xacro:wamv_ball_shooter name="ball_shooter" x="0.55" y="-0.3" z="1.3" pitch="${radians(-20)}" yaw="0" />
+    <!-- === wamv_pinger === -->
+      <xacro:wamv_pinger sensor_name="receiver" position="1.0 0 -1.0" />
   </xacro:macro>
 </robot>

File: utils/vrx/x_drive/usv.urdf (robot description, URDF)
Before this commit: robot WAM-V, 31 links, 30 joints
Links:
- added link wamv/receiver, mass 0.1; visual sphere radius=0.01
Joints:
- added joint wamv/receiver_pinger_joint: type revolute, parent wamv/base_link, child wamv/receiver, origin xyz=0 0 0 rpy=0 0 0, axis 0 0 1, limit lower=0.0 upper=0 effort=1000.0 velocity=0
