Commit message: h drive urdf

File: utils/roboboat/h_drive/usv.urdf (robot description, URDF)
Before this commit: robot WAM-V, 36 links, 35 joints
Links:
- link wamv/lidar_wamv_post_arm_link: geometry 
- link wamv/lidar_wamv_post_link: mass 0.40815000000000007 -> -0.76185; geometry 
Joints:
- joint wamv/base_to_lidar_wamv_post_joint: origin xyz=0.6299999999999999 0.0 1.52325 rpy=0 0 0 -> xyz=2.43 0.0 0.87325 rpy=0 0 0
- joint wamv/front_left_camera_post_arm_to_front_left_camera_joint: origin xyz=0.02 0 0.027 rpy=0 0.2617993877991494 0 -> xyz=0.02 0 0.027 rpy=0 0 0
- joint wamv/front_right_camera_post_arm_to_front_right_camera_joint: origin xyz=0.02 0 0.027 rpy=0 0.2617993877991494 0 -> xyz=0.02 0 0.027 rpy=0 0 0
- joint wamv/lidar_wamv_post_arm_to_lidar_wamv_joint: origin xyz=0.04 0 0.05 rpy=0 0.13962634015954636 0 -> xyz=0.04 0 0.05 rpy=0 0 0
- joint wamv/lidar_wamv_post_to_lidar_wamv_post_arm_joint: origin xyz=0.03 0 0.22675000000000006 rpy=0 0 0 -> xyz=0.03 0 -0.42324999999999996 rpy=0 0 0
- joint wamv/middle_right_camera_post_arm_to_middle_right_camera_joint: origin xyz=0.02 0 0.027 rpy=0 0.2617993877991494 0 -> xyz=0.02 0 0.027 rpy=0 0 0

Commit message: nav2_costmap fail

File: utils/roboboat/h_drive/usv.urdf (robot description, URDF)
Before this commit: robot WAM-V, 36 links, 35 joints
Links:
- removed link wamv/dummy_link
- link wamv/base_link: mass None -> 180.0; geometry collision box size=0.65 0.2 0.1; collision box size=0.65 0.2 0.1
- link wamv/imu_wamv_link: geometry collision box size=0.05 0.025 0.005; visual box size=0.05 0.025 0.005
- link wamv/lidar_wamv_post_arm_link: geometry collision cylinder length=0.065 radius=0.008; visual mesh filename=package://vrx_gazebo/models/sensor_post/mesh/sensor_post_ar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
- link wamv/lidar_wamv_post_link: mass -0.76185 -> 0.40815000000000007; geometry collision cylinder length=0.45350000000000007 radius=0.0076; visual cylinder length=0.45350000000000007 radius=0.0076
Joints:
- removed joint wamv/dummy_joint
- removed joint wamv/left_front_chasis_engine_joint
- removed joint wamv/left_middle_chasis_engine_joint
- removed joint wamv/left_rear_chasis_engine_joint
- removed joint wamv/right_front_chasis_engine_joint
- removed joint wamv/right_middle_chasis_engine_joint
- removed joint wamv/right_rear_chasis_engine_joint
- added joint wamv/left_front_chassis_engine_joint: type revolute, parent wamv/base_link, child wamv/left_front_engine_link, origin xyz=1.6 0.7 0.25 rpy=0.0 0.0 -0.785, axis 0 0 1, limit lower=-3.141592653589793 upper=3.141592653589793 effort=10 velocity=10
- added joint wamv/left_middle_chassis_engine_joint: type revolute, parent wamv/base_link, child wamv/left_middle_engine_link, origin xyz=0 0.7 0.25 rpy=0.0 0.0 -1.5708, axis 0 0 1, limit lower=-3.141592653589793 upper=3.141592653589793 effort=10 velocity=10
- added joint wamv/left_rear_chassis_engine_joint: type revolute, parent wamv/base_link, child wamv/left_rear_engine_link, origin xyz=-2.373776 1.027135 0.318237 rpy=0.0 0.0 0.785, axis 0 0 1, limit lower=-3.141592653589793 upper=3.141592653589793 effort=10 velocity=10
- added joint wamv/right_front_chassis_engine_joint: type revolute, parent wamv/base_link, child wamv/right_front_engine_link, origin xyz=1.6 -0.7 0.25 rpy=0.0 0.0 0.785, axis 0 0 1, limit lower=-3.141592653589793 upper=3.141592653589793 effort=10 velocity=10
- added joint wamv/right_middle_chassis_engine_joint: type revolute, parent wamv/base_link, child wamv/right_middle_engine_link, origin xyz=0 -0.7 0.25 rpy=0.0 0.0 1.5708, axis 0 0 1, limit lower=-3.141592653589793 upper=3.141592653589793 effort=10 velocity=10
- added joint wamv/right_rear_chassis_engine_joint: type revolute, parent wamv/base_link, child wamv/right_rear_engine_link, origin xyz=-2.373776 -1.027135 0.318237 rpy=0.0 0.0 -0.785, axis 0 0 1, limit lower=-3.141592653589793 upper=3.141592653589793 effort=10 velocity=10
- joint wamv/base_to_lidar_wamv_post_joint: origin xyz=2.43 0.0 0.87325 rpy=0 0 0 -> xyz=0.6299999999999999 -0.3 1.52325 rpy=0 0 0
- joint wamv/lidar_wamv_post_to_lidar_wamv_post_arm_joint: origin xyz=0.03 0 -0.42324999999999996 rpy=0 0 0 -> xyz=0.03 0 0.22675000000000006 rpy=0 0 0
